Commit message: remove collision leg

File: spot_description/urdf/spot_leg.urdf.xacro (robot description, xacro)
@@ -31,5 +31,5 @@
                 </geometry>
             </visual>
-            <collision>
+            <!-- <collision>
                 <origin rpy="0 0 0" xyz="0 0 0"/>
                 <geometry>
@@ -37,5 +37,5 @@
                     <cylinder radius="${hip_width}" length="${hip_length}"/>
                 </geometry>
-            </collision>
+            </collision> -->
             <inertial>
                 <mass value="${hip_mass}"/>
@@ -69,5 +69,5 @@
                 <origin rpy="0 0 0" xyz="0 0 ${-0.25*upper_leg_height}"/>
                 <geometry>
-                    <mesh filename="package://spot_description/meshes/${leg_name}_upper_leg_collision.stl" />
+                    <!-- <mesh filename="package://spot_description/meshes/${leg_name}_upper_leg_collision.stl" /> -->
                     <cylinder radius="${0.6*upper_leg_width}" length="${0.8*upper_leg_height}"/>
                 </geometry>
@@ -105,5 +105,5 @@
                 <origin rpy="0 0 0" xyz="0 0 ${-0.35*lower_leg_height}"/>
                 <geometry>
-                    <mesh filename="package://spot_description/meshes/${leg_name_long}_lower_leg_collision.stl" scale="0.82 0.97 0.98"/>
+                    <!-- <mesh filename="package://spot_description/meshes/${leg_name_long}_lower_leg_collision.stl" scale="0.82 0.97 0.98"/> -->
                     <cylinder radius="${lower_leg_length}" length="${0.6*lower_leg_height}"/>
                 </geometry>
@@ -136,5 +136,5 @@
                 <origin rpy="0 0 0" xyz="0 0 ${lower_leg_length}"/>
                 <geometry>
-                    <mesh filename="package://spot_description/meshes/${leg_name_long}_lower_leg_collision.stl" scale="0.82 0.97 0.98"/>
+                    <!-- <mesh filename="package://spot_description/meshes/${leg_name_long}_lower_leg_collision.stl" scale="0.82 0.97 0.98"/> -->
                     <sphere radius="${lower_leg_length}"/>
                 </geometry>
