Commit message: test

File: go2w_description/urdf/go2w_description.urdf (robot description, URDF)
Before this commit: robot go2w_description, 33 links, 32 joints
Joints:
- joint RR_calf_joint: axis 0 1 0 -> 1 0 0

Commit message: test2

File: go2w_description/urdf/go2w_description.urdf (robot description, URDF)
Before this commit: robot go2w_description, 33 links, 32 joints
Joints:
- joint RR_calf_joint: axis 1 0 0 -> 0 0 1

Commit message: Test

File: go2w_description/urdf/go2w_description.urdf (robot description, URDF)
Before this commit: robot go2w_description, 33 links, 32 joints
Joints:
- joint RR_calf_joint: axis 0 0 1 -> 0 1 0; origin xyz=0 0 -0.213 rpy=0 0 0 -> xyz=0 0 -0.213 rpy=1.5707963267948966 0 0

Commit message: Test

File: go2w_description/urdf/go2w_description.urdf (robot description, URDF)
Before this commit: robot go2w_description, 33 links, 32 joints
Joints:
- joint RR_calf_joint: origin xyz=0 0 -0.213 rpy=1.5707963267948966 0 0 -> xyz=0 0 -0.213 rpy=0 1.5707963267948966 0

Commit message: argh

File: go2w_description/urdf/go2w_description.urdf (robot description, URDF)
Before this commit: robot go2w_description, 33 links, 32 joints
Joints:
- joint RR_calf_joint: origin xyz=0 0 -0.213 rpy=0 1.5707963267948966 0 -> xyz=0 0 -0.213 rpy=0 0 1.5707963267948966

Commit message: test

File: go2w_description/urdf/go2w_description.urdf (robot description, URDF)
Before this commit: robot go2w_description, 33 links, 32 joints
Joints:
- joint RR_calf_joint: origin xyz=0 0 -0.213 rpy=0 0 1.5707963267948966 -> xyz=0 0 -0.213 rpy=0 0 0
