Commit message: fix xacro

File: b2w_description/xacro/robot.urdf.xacro (robot description, xacro)
@@ -6,4 +6,18 @@
   xmlns:controller="http://playerstage.sourceforge.net/gazebo/xmlschema/#controller"
   xmlns:interface="http://playerstage.sourceforge.net/gazebo/xmlschema/#interface" >
-  <xacro:include filename="$(find b2w_description)/urdf/b2w_description.urdf"/>
+  <link name="base_link"/>
+  <joint
+    name="base_link_joint"
+    type="fixed" dont_collapse="true">
+    <origin
+      xyz="0 0 0"
+      rpy="0 0 0" />
+    <parent
+      link="base_link" />
+    <child
+      link="base" />
+    <axis
+      xyz="0 0 0" />
+  </joint>
+  <xacro:include filename="package://b2w_description/urdf/b2w_description.urdf" />
 </robot>
