Commit message: replace relative paths

File: m20_description/urdf/M20.urdf (robot description, URDF)
Before this commit: robot M20, 17 links, 16 joints
Links:
- link base_link: geometry collision box size=0.75 0.09 0.14; collision cylinder length=0.75 radius=0.07
- link fl_hipx: geometry collision cylinder length=0.14 radius=0.048; visual mesh filename=package://m20_description/meshes/fl_hipx.STL
- link fl_hipy: geometry collision box size=0.07 0.02 0.25; collision cylinder length=0.09 radius=0.05
- link fl_knee: geometry collision box size=0.06 0.025 0.25; collision cylinder length=0.1 radius=0.04
- link fl_wheel: geometry collision cylinder length=0.054 radius=0.09; visual mesh filename=package://m20_description/meshes/fl_wheel.STL
- link fr_hipx: geometry collision cylinder length=0.14 radius=0.048; visual mesh filename=package://m20_description/meshes/fr_hipx.STL
- link fr_hipy: geometry collision box size=0.07 0.02 0.25; collision cylinder length=0.09 radius=0.05
- link fr_knee: geometry collision box size=0.06 0.025 0.25; collision cylinder length=0.1 radius=0.04
- link fr_wheel: geometry collision cylinder length=0.054 radius=0.09; visual mesh filename=package://m20_description/meshes/fr_wheel.STL
- link hl_hipx: geometry collision cylinder length=0.14 radius=0.048; visual mesh filename=package://m20_description/meshes/hl_hipx.STL
- link hl_hipy: geometry collision box size=0.07 0.02 0.25; collision cylinder length=0.09 radius=0.05
- link hl_knee: geometry collision box size=0.06 0.025 0.25; collision cylinder length=0.1 radius=0.04
- link hl_wheel: geometry collision cylinder length=0.054 radius=0.09; visual mesh filename=package://m20_description/meshes/hl_wheel.STL
- link hr_hipx: geometry collision cylinder length=0.14 radius=0.048; visual mesh filename=package://m20_description/meshes/hr_hipx.STL
- link hr_hipy: geometry collision box size=0.07 0.02 0.25; collision cylinder length=0.09 radius=0.05
- link hr_knee: geometry collision box size=0.06 0.025 0.25; collision cylinder length=0.1 radius=0.04
- link hr_wheel: geometry collision cylinder length=0.054 radius=0.09; visual mesh filename=package://m20_description/meshes/hr_wheel.STL

File: x30_description/urdf/X30.urdf (robot description, URDF)
Before this commit: robot X30, 17 links, 16 joints
Links:
- link FL_HIP: geometry visual mesh filename=package://x30_description/meshes/hip.STL
- link FL_SHANK: geometry collision cylinder length=0.08 radius=0.015; collision cylinder length=0.1 radius=0.015
- link FL_THIGH: geometry collision cylinder length=0.25 radius=0.04; visual mesh filename=package://x30_description/meshes/thigh.STL
- link FR_HIP: geometry visual mesh filename=package://x30_description/meshes/hip.STL scale=1 -1 1
- link FR_SHANK: geometry collision cylinder length=0.08 radius=0.015; collision cylinder length=0.1 radius=0.015
- link FR_THIGH: geometry collision cylinder length=0.25 radius=0.04; visual mesh filename=package://x30_description/meshes/thigh.STL scale=1 -1 1
- link HL_HIP: geometry visual mesh filename=package://x30_description/meshes/hip.STL scale=-1 1 1
- link HL_SHANK: geometry collision cylinder length=0.08 radius=0.015; collision cylinder length=0.1 radius=0.015
- link HL_THIGH: geometry collision cylinder length=0.25 radius=0.04; visual mesh filename=package://x30_description/meshes/thigh.STL
- link HR_HIP: geometry visual mesh filename=package://x30_description/meshes/hip.STL scale=-1 -1 1
- link HR_SHANK: geometry collision cylinder length=0.08 radius=0.015; collision cylinder length=0.1 radius=0.015
- link HR_THIGH: geometry collision cylinder length=0.25 radius=0.04; visual mesh filename=package://x30_description/meshes/thigh.STL scale=1 -1 1
- link TORSO: geometry collision box size=0.46 0.26 0.18; visual mesh filename=package://x30_description/meshes/torso.STL
